File: GPS.sch (KiCad schematic (older format))
At the start: 8 parts, among them J10 SMAConn, SW3 GPS_BattCheck, U7 MTK3339

Commit message: Adds phy resistors and moves power conn away from recom
Parts:
- U7: symbol utsvt-chips:MTK3339 -> Telemetry-Primary-rescue:MTK3339-utsvt-chips
Changed lines of the file:
@@
 $EndComp
 $Comp
-L utsvt-chips:MTK3339 U7
+L Telemetry-Primary-rescue:MTK3339-utsvt-chips U7
 U 1 1 5FB7A882
 P 4700 3650
