File: RTCC.sch (KiCad schematic (older format))
At the start: 8 parts, among them SW2 RTCC_BattCheck, U6 PCF8523T, Y3 32.768k

Commit message: Adds phy resistors and moves power conn away from recom
Parts:
- U6: symbol Telemetry-Primary-rescue:PCF8523T-Timer_RTC -> Telemetry-Primary-rescue:PCF8523T-Timer_RTC-Telemetry-Primary-rescue
Changed lines of the file:
@@
 $EndDescr
 $Comp
-L Telemetry-Primary-rescue:PCF8523T-Timer_RTC U6
+L Telemetry-Primary-rescue:PCF8523T-Timer_RTC-Telemetry-Primary-rescue U6
 U 1 1 5F6F240B
 P 5000 3750
