File: SDCard.sch (KiCad schematic (older format))
At the start: 1 part, among them J9 Micro_SD_Card_Det

Commit message: Adds phy resistors and moves power conn away from recom
Parts:
- J9: symbol Telemetry-Primary-rescue:Micro_SD_Card_Det-Connector -> Telemetry-Primary-rescue:Micro_SD_Card_Det-Connector-Telemetry-Primary-rescue
Changed lines of the file:
@@
 	4550 3600 3950 3600
 $Comp
-L Telemetry-Primary-rescue:Micro_SD_Card_Det-Connector J9
+L Telemetry-Primary-rescue:Micro_SD_Card_Det-Connector-Telemetry-Primary-rescue J9
 U 1 1 5F718A2C
 P 5450 3900
