File: USB.sch (KiCad schematic (older format))
At the start: 8 parts, among them J11 USB_B_Micro, U9 CP2102N-A01-GQFN24

Commit message: Adds phy resistors and moves power conn away from recom
Parts:
- D5: symbol Telemetry-Primary-rescue:SP0503BAHT-Power_Protection -> Telemetry-Primary-rescue:SP0503BAHT-Power_Protection-Telemetry-Primary-rescue
- J11: symbol Telemetry-Primary-rescue:USB_B_Micro-Connector -> Telemetry-Primary-rescue:USB_B_Micro-Connector-Telemetry-Primary-rescue
Changed lines of the file:
@@
 $EndComp
 $Comp
-L Telemetry-Primary-rescue:USB_B_Micro-Connector J11
+L Telemetry-Primary-rescue:USB_B_Micro-Connector-Telemetry-Primary-rescue J11
 U 1 1 5C4964BB
 P 3000 4300
@@
 	5500 4750 5500 4800
 $Comp
-L Telemetry-Primary-rescue:SP0503BAHT-Power_Protection D5
+L Telemetry-Primary-rescue:SP0503BAHT-Power_Protection-Telemetry-Primary-rescue D5
 U 1 1 5C496C9B
 P 3950 4800
