File: CAN.kicad_sch (KiCad schematic)
At the start: 19 parts, among them J12 CAN_In, J13 CAN_Out, U10 ADM3055E, U11 CDSOT23-T24CAN

Commit message: bom, gerbers, edge cuts, footprint verification
Parts:
- C42, C47: P/N (none) -> 0805YC106KAT2A
- C43, C44, C48: P/N (none) -> C0805C104K5RAC7411
- C45, C49: P/N (none) -> AC0805JRX7R9BB103
- C46: P/N (none) -> C0805C224K1RECAUTO
- J12, J13: P/N (none) -> 0436500428
- JP1: P/N (none) -> 10129378-910001BLF
- L1, L2: P/N (none) -> MMZ2012Y202BTD25
- R34: P/N (none) -> CRCW08050000Z0EAC
- R35: P/N (none) -> CRCW0805120RFKEAC
- TP6, TP7: P/N (none) -> 5005
- U10: P/N (none) -> ADM3055EBRIZ
- U11: P/N (none) -> CDSOT23-T24CAN
Changed lines of the file:
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@@
       (effects (font (size 1.524 1.524)) hide)
     )
-    (property "Datasheet" "" (at 245.11 88.9 0)
-      (effects (font (size 1.524 1.524)) hide)
+    (property "Datasheet" "https://www.mouser.com/datasheet/2/276/3/0436500428_PCB_HEADERS-2866587.pdf" (at 245.11 88.9 0)
+      (effects (font (size 1.524 1.524)) hide)
+    )
+    (property "P/N" "0436500428" (at 248.92 96.52 0)
+      (effects (font (size 1.27 1.27)) hide)
     )
     (pin "1")
@@
       (effects (font (size 1.27 1.27)) hide)
     )
-    (property "Datasheet" "~" (at 200.66 109.22 0)
+    (property "Datasheet" "https://www.mouser.com/datasheet/2/427/dcrcwe3-1762152.pdf" (at 200.66 109.22 0)
+      (effects (font (size 1.27 1.27)) hide)
+    )
+    (property "P/N" "CRCW0805120RFKEAC" (at 200.66 109.22 0)
       (effects (font (size 1.27 1.27)) hide)
     )
@@
       (effects (font (size 1.27 1.27)) hide)
     )
-    (property "Datasheet" "~" (at 54.61 85.09 0)
+    (property "Datasheet" "https://www.mouser.com/datasheet/2/40/AVX_X7RDielectric_777024-1853642.pdf" (at 54.61 85.09 0)
+      (effects (font (size 1.27 1.27)) hide)
+    )
+    (property "P/N" "0805YC106KAT2A" (at 54.61 85.09 0)
       (effects (font (size 1.27 1.27)) hide)
     )
@@
       (effects (font (size 1.27 1.27)) hide)
     )
-    (property "Datasheet" "~" (at 63.5 85.09 0)
+    (property "Datasheet" "https://www.mouser.com/datasheet/2/212/KEM_C1002_X7R_SMD-1102033.pdf" (at 63.5 85.09 0)
+      (effects (font (size 1.27 1.27)) hide)
+    )
+    (property "P/N" "C0805C104K5RAC7411" (at 63.5 85.09 0)
       (effects (font (size 1.27 1.27)) hide)
     )
@@
       (effects (font (size 1.27 1.27)) hide)
     )
-    (property "Datasheet" "~" (at 74.93 85.09 0)
+    (property "Datasheet" "https://www.mouser.com/datasheet/2/212/KEM_C1002_X7R_SMD-1102033.pdf" (at 74.93 85.09 0)
+      (effects (font (size 1.27 1.27)) hide)
+    )
+    (property "P/N" "C0805C104K5RAC7411" (at 74.93 85.09 0)
       (effects (font (size 1.27 1.27)) hide)
     )
@@
       (effects (font (size 1.27 1.27)) hide)
     )
-    (property "Datasheet" "~" (at 83.82 85.09 0)
+    (property "Datasheet" "https://www.mouser.com/datasheet/2/447/UPY_AC_NP0X7RX7S_6_3V_to_2KV_18-3003021.pdf" (at 83.82 85.09 0)
+      (effects (font (size 1.27 1.27)) hide)
+    )
+    (property "P/N" "AC0805JRX7R9BB103" (at 83.82 85.09 0)
       (effects (font (size 1.27 1.27)) hide)
     )
@@
       (effects (font (size 1.27 1.27)) hide)
     )
-    (property "Datasheet" "~" (at 156.21 81.28 0)
+    (property "Datasheet" "https://www.mouser.com/datasheet/2/40/AVX_X7RDielectric_777024-1853642.pdf" (at 156.21 81.28 0)
+      (effects (font (size 1.27 1.27)) hide)
+    )
+    (property "P/N" "0805YC106KAT2A" (at 156.21 81.28 0)
       (effects (font (size 1.27 1.27)) hide)
     )
@@
       (effects (font (size 1.27 1.27)) hide)
     )
-    (property "Datasheet" "~" (at 146.05 81.28 0)
+    (property "Datasheet" "https://www.mouser.com/datasheet/2/212/1/KEM_C1090_X7R_ESD-1103328.pdf" (at 146.05 81.28 0)
+      (effects (font (size 1.27 1.27)) hide)
+    )
+    (property "P/N" "C0805C224K1RECAUTO" (at 146.05 81.28 0)
       (effects (font (size 1.27 1.27)) hide)
     )
@@
       (effects (font (size 1.27 1.27)) hide)
     )
-    (property "Datasheet" "https://product.tdk.com/info/en/catalog/datasheets/beads_commercial_signal_mmz2012_en.pdf?ref_disty=mouser" (at 151.13 77.47 0)
+    (property "Datasheet" "https://product.tdk.com/system/files/dam/doc/product/emc/emc/beads/catalog/beads_automotive_signal_mmz2012_en.pdf" (at 151.13 77.47 0)
+      (effects (font (size 1.27 1.27)) hide)
+    )
+    (property "P/N" "MMZ2012Y202BTD25" (at 151.13 77.47 0)
       (effects (font (size 1.27 1.27)) hide)
     )
@@
       (effects (font (size 1.27 1.27)) hide)
     )
-    (property "Datasheet" "https://product.tdk.com/info/en/catalog/datasheets/beads_commercial_signal_mmz2012_en.pdf?ref_disty=mouser" (at 151.13 85.09 0)
+    (property "Datasheet" "https://product.tdk.com/system/files/dam/doc/product/emc/emc/beads/catalog/beads_automotive_signal_mmz2012_en.pdf" (at 151.13 85.09 0)
+      (effects (font (size 1.27 1.27)) hide)
+    )
+    (property "P/N" "MMZ2012Y202BTD25" (at 151.13 85.09 0)
       (effects (font (size 1.27 1.27)) hide)
     )
@@
       (effects (font (size 1.27 1.27)) hide)
     )
-    (property "Datasheet" "~" (at 166.37 81.28 0)
+    (property "Datasheet" "https://www.mouser.com/datasheet/2/212/KEM_C1002_X7R_SMD-1102033.pdf" (at 166.37 81.28 0)
+      (effects (font (size 1.27 1.27)) hide)
+    )
+    (property "P/N" "C0805C104K5RAC7411" (at 166.37 81.28 0)
       (effects (font (size 1.27 1.27)) hide)
     )
@@
       (effects (font (size 1.27 1.27)) hide)
     )
-    (property "Datasheet" "~" (at 173.99 81.28 0)
+    (property "Datasheet" "https://www.mouser.com/datasheet/2/447/UPY_AC_NP0X7RX7S_6_3V_to_2KV_18-3003021.pdf" (at 173.99 81.28 0)
+      (effects (font (size 1.27 1.27)) hide)
+    )
+    (property "P/N" "AC0805JRX7R9BB103" (at 173.99 81.28 0)
       (effects (font (size 1.27 1.27)) hide)
     )
@@
       (effects (font (size 1.524 1.524)) hide)
     )
-    (property "Datasheet" "" (at 110.49 88.9 0)
-      (effects (font (size 1.524 1.524)) hide)
+    (property "Datasheet" "https://www.mouser.com/datasheet/2/609/ADM3055E_3057E-3121303.pdf" (at 110.49 88.9 0)
+      (effects (font (size 1.524 1.524)) hide)
+    )
+    (property "P/N" "ADM3055EBRIZ" (at 110.49 91.44 0)
+      (effects (font (size 1.27 1.27)) hide)
     )
     (pin "1")
@@
       (effects (font (size 1.524 1.524)) hide)
     )
-    (property "Datasheet" "https://www.mouser.com/datasheet/2/54/cdsot23-t24can-q-1534349.pdf" (at 205.74 88.9 0)
-      (effects (font (size 1.524 1.524)) hide)
+    (property "Datasheet" "https://www.mouser.com/datasheet/2/54/cdsot23_t24can_q-1534349.pdf" (at 205.74 88.9 0)
+      (effects (font (size 1.524 1.524)) hide)
+    )
+    (property "P/N" "CDSOT23-T24CAN" (at 205.74 88.9 0)
+      (effects (font (size 1.27 1.27)) hide)
     )
     (pin "1")
@@
       (effects (font (size 1.27 1.27)) hide)
     )
-    (property "Datasheet" "~" (at 185.42 96.52 0)
+    (property "Datasheet" "https://www.mouser.com/datasheet/2/215/5005_5009-741322.pdf" (at 185.42 96.52 0)
+      (effects (font (size 1.27 1.27)) hide)
+    )
+    (property "P/N" "5005" (at 185.42 96.52 0)
       (effects (font (size 1.27 1.27)) hide)
     )
@@
       (effects (font (size 1.27 1.27)) hide)
     )
-    (property "Datasheet" "~" (at 185.42 101.6 0)
+    (property "Datasheet" "https://www.mouser.com/datasheet/2/215/5005_5009-741322.pdf" (at 185.42 101.6 0)
+      (effects (font (size 1.27 1.27)) hide)
+    )
+    (property "P/N" "5005" (at 185.42 101.6 0)
       (effects (font (size 1.27 1.27)) hide)
     )
@@
       (effects (font (size 1.27 1.27)) hide)
     )
-    (property "Datasheet" "~" (at 140.97 105.41 0)
+    (property "Datasheet" "https://www.mouser.com/datasheet/2/427/dcrcwe3-1762152.pdf" (at 140.97 105.41 0)
+      (effects (font (size 1.27 1.27)) hide)
+    )
+    (property "P/N" "CRCW08050000Z0EAC" (at 140.97 105.41 0)
       (effects (font (size 1.27 1.27)) hide)
     )
@@
       (effects (font (size 1.524 1.524)) hide)
     )
-    (property "Datasheet" "" (at 245.11 72.39 0)
-      (effects (font (size 1.524 1.524)) hide)
+    (property "Datasheet" "https://www.mouser.com/datasheet/2/276/3/0436500428_PCB_HEADERS-2866587.pdf" (at 245.11 72.39 0)
+      (effects (font (size 1.524 1.524)) hide)
+    )
+    (property "P/N" "0436500428" (at 248.92 80.01 0)
+      (effects (font (size 1.27 1.27)) hide)
     )
     (pin "1")
@@
       (effects (font (size 1.27 1.27)) hide)
     )
-    (property "Datasheet" "https://cdn.amphenol-icc.com/media/wysiwyg/files/documentation/datasheet/boardwiretoboard/bwb_econostik_254headers.pdf" (at 210.82 109.22 0)
-      (effects (font (size 1.27 1.27)) hide)
-    )
+    (property "Datasheet" "https://cdn.amphenol-cs.com/media/wysiwyg/files/documentation/datasheet/boardwiretoboard/bwb_econostik_254headers.pdf" (at 210.82 109.22 0)
+      (effects (font (size 1.27 1.27)) hide)
+    )
+    (property "P/N" "10129378-910001BLF" (at 210.82 109.22 0)
+      (effects (font (size 1.27 1.27)) hide)
+    )
