File: IMU.kicad_sch (KiCad schematic)
At the start: 8 parts

Commit message: bom, gerbers, edge cuts, footprint verification
Parts:
- C36: P/N (none) -> C0805F682K1RACAUTO
- C37: P/N (none) -> 08053C124JAT2A
- C38: P/N (none) -> C0805C104K5RAC7411
- C39: value 100n -> 0.1u; P/N (none) -> C0805C104K5RAC7411
- R28, R29, R30: P/N (none) -> CRCW080510K0FKEAC
- U?: P/N (none) -> BNO055
Changed lines of the file:
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@@
       (effects (font (size 1.27 1.27)) (justify left) hide)
     )
-    (property "Datasheet" "https://ae-bst.resource.bosch.com/media/_tech/media/datasheets/BST_BNO055_DS000_14.pdf" (at 160.02 91.44 0)
+    (property "Datasheet" "https://www.mouser.com/datasheet/2/783/BST_BNO055_DS000-1509603.pdf" (at 160.02 91.44 0)
+      (effects (font (size 1.27 1.27)) hide)
+    )
+    (property "P/N" "BNO055" (at 160.02 96.52 0)
       (effects (font (size 1.27 1.27)) hide)
     )
@@
   (symbol (lib_id "Device:C") (at 181.61 109.22 270) (unit 1)
     (in_bom yes) (on_board yes) (dnp no)
-    (property "Reference" "C38" (at 184.15 110.49 90)
+    (property "Reference" "C38" (at 184.785 110.49 90)
       (effects (font (size 1.27 1.27)))
     )
@@
       (effects (font (size 1.27 1.27)) hide)
     )
-    (property "Datasheet" "~" (at 181.61 109.22 0)
+    (property "Datasheet" "https://www.mouser.com/datasheet/2/212/KEM_C1002_X7R_SMD-1102033.pdf" (at 181.61 109.22 0)
+      (effects (font (size 1.27 1.27)) hide)
+    )
+    (property "P/N" "C0805C104K5RAC7411" (at 181.61 109.22 0)
       (effects (font (size 1.27 1.27)) hide)
     )
@@
   (symbol (lib_id "Device:R") (at 134.62 76.2 0) (unit 1)
     (in_bom yes) (on_board yes) (dnp no)
-    (property "Reference" "R28" (at 136.398 75.0316 0)
-      (effects (font (size 1.27 1.27)) (justify left))
-    )
-    (property "Value" "10k" (at 136.398 77.343 0)
+    (property "Reference" "R28" (at 135.89 74.93 0)
+      (effects (font (size 1.27 1.27)) (justify left))
+    )
+    (property "Value" "10k" (at 135.89 77.47 0)
       (effects (font (size 1.27 1.27)) (justify left))
     )
@@
       (effects (font (size 1.27 1.27)) hide)
     )
-    (property "Datasheet" "~" (at 134.62 76.2 0)
+    (property "Datasheet" "https://www.mouser.com/datasheet/2/427/dcrcwe3-1762152.pdf" (at 134.62 76.2 0)
+      (effects (font (size 1.27 1.27)) hide)
+    )
+    (property "P/N" "CRCW080510K0FKEAC" (at 134.62 76.2 0)
       (effects (font (size 1.27 1.27)) hide)
     )
@@
       (effects (font (size 1.27 1.27)) hide)
     )
-    (property "Datasheet" "~" (at 104.14 99.06 0)
+    (property "Datasheet" "https://www.mouser.com/datasheet/2/40/X7RDielectric-2943470.pdf" (at 104.14 99.06 0)
+      (effects (font (size 1.27 1.27)) hide)
+    )
+    (property "P/N" "08053C124JAT2A" (at 104.14 99.06 0)
       (effects (font (size 1.27 1.27)) hide)
     )
@@
       (effects (font (size 1.27 1.27)) (justify left))
     )
-    (property "Value" "100n" (at 192.151 98.933 0)
+    (property "Value" "0.1u" (at 192.151 98.933 0)
       (effects (font (size 1.27 1.27)) (justify left))
     )
@@
       (effects (font (size 1.27 1.27)) hide)
     )
-    (property "Datasheet" "~" (at 189.23 97.79 0)
+    (property "Datasheet" "https://www.mouser.com/datasheet/2/212/KEM_C1002_X7R_SMD-1102033.pdf" (at 189.23 97.79 0)
+      (effects (font (size 1.27 1.27)) hide)
+    )
+    (property "P/N" "C0805C104K5RAC7411" (at 189.23 97.79 0)
       (effects (font (size 1.27 1.27)) hide)
     )
@@
       (effects (font (size 1.27 1.27)) hide)
     )
-    (property "Datasheet" "~" (at 140.97 76.2 0)
+    (property "Datasheet" "https://www.mouser.com/datasheet/2/427/dcrcwe3-1762152.pdf" (at 140.97 76.2 0)
+      (effects (font (size 1.27 1.27)) hide)
+    )
+    (property "P/N" "CRCW080510K0FKEAC" (at 140.97 76.2 0)
       (effects (font (size 1.27 1.27)) hide)
     )
@@
       (effects (font (size 1.27 1.27)) hide)
     )
-    (property "Datasheet" "~" (at 135.89 109.22 0)
+    (property "Datasheet" "https://www.mouser.com/datasheet/2/427/dcrcwe3-1762152.pdf" (at 135.89 109.22 0)
+      (effects (font (size 1.27 1.27)) hide)
+    )
+    (property "P/N" "CRCW080510K0FKEAC" (at 135.89 109.22 0)
       (effects (font (size 1.27 1.27)) hide)
     )
@@
       (effects (font (size 1.27 1.27)) hide)
     )
-    (property "Datasheet" "~" (at 91.44 104.14 0)
-      (effects (font (size 1.27 1.27)) hide)
-    )
+    (property "Datasheet" "https://www.mouser.com/datasheet/2/212/KEM_C1012_X7R_OPENMODE_SMD-1103265.pdf" (at 91.44 104.14 0)
+      (effects (font (size 1.27 1.27)) hide)
+    )
+    (property "P/N" "C0805F682K1RACAUTO" (at 91.44 104.14 0)
+      (effects (font (size 1.27 1.27)) hide)
+    )
