File: Telemetry-Primary.kicad_sch (KiCad schematic)
At the start: 39 parts, among them J1 CAN_LogicAnalyzer, J2 IMU_LogicAnalyzer, J3 GPS_LogicAnalyzer, J4 RTCC_LogicAnalyzer, J5 SDCard_LogicAnalyzer, J6 SWD, SW1 Reset, U1 STM32F429ZITx, Y1 8M

Commit message: merged v2.1 changes
removes external RTC, cleaned up big errors, only minor warnings remain
Parts:
- removed J4: RTCC_LogicAnalyzer, Connector_PinHeader_2.54mm:PinHeader_1x04_P2.54mm_Vertical, symbol Connector_Generic:Conn_01x04
- removed R? (x2): 4.7k, Resistor_SMD:R_0805_2012Metric, symbol Device:R
- added BT?: CR1220, Battery:BatteryHolder_Keystone_3000_1x12mm, symbol Device:Battery_Cell
- added C35, C50: 9p, Capacitor_SMD:C_0805_2012Metric, symbol Device:C_Small
- added D?: RTCC_BattCheck, LED_SMD:LED_0805_2012Metric, symbol Device:LED_Small
- added R?: 550, Resistor_SMD:R_0805_2012Metric, symbol Device:R_Small
- added SW?: RTCC_BattCheck, Button_Switch_SMD:SW_SPST_B3SL-1002P, symbol Switch:SW_Push
- added Y3: 32.768k, Crystal:Crystal_SMD_2012-2Pin_2.0x1.2mm, symbol Device:Crystal_Small
Connections:
- net +3.3V: no longer C9.1, U1.6 (VBAT)
- net GND: now also BT?.2 (-), C35.1, C50.1, SW?.2
- net at U1.8 (PC14): now also C35.2, Y3.1
- net at U1.9 (PC15): now also C50.2, Y3.2
- net I2C2_SCL: no longer names the net of U1.69 (PB10)
- net I2C2_SDA: no longer names the net of U1.70 (PB11)
- net PB12: no longer names the net of U1.73 (PB12)
- net USART2_RX: no longer names the net of U1.122 (PD6)
- net USART2_TX: no longer names the net of U1.119 (PD5)
- new net: D?.1 (K), SW?.1
- new net: D?.2 (A), R?.2
- new net +BATT: BT?.1 (+), C9.1, R?.1, U1.6 (VBAT)
- no-connect marks 74 -> 75
Other:
- removed sheet RTCC
- note added: "Check levels of coin cell battery without having the led constantly consume power."
- note added: "Version History -v2.1, Remove the external RTC. There's no need to use an external RTC on the telemetry board. The microcontroller itself has an internal RTC that can be powered from the VBAT line and a 32.768kHz oscillator. Courtesy of Chase!"
- note removed: "Addr: 0x68"
- moved on the sheet: C11, C12, C13, C14, C15, C16, C17, C18, C19, C20, C5, C7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

Commit message: cleaner, still needs full checklisting
Parts:
- SW1, SW?: footprint Button_Switch_SMD:SW_SPST_B3SL-1002P -> UTSVT_Special:SW_SPST_B3SL-1002P
- Y1: footprint Crystal:Crystal_SMD_TXC_7A-2Pin_5x3.2mm -> UTSVT_Special:Crystal_SMD_TXC_7A-2Pin_5x3.2mm
- Y3: footprint Crystal:Crystal_SMD_2012-2Pin_2.0x1.2mm -> UTSVT_Special:Crystal_SMD_2012-2Pin_2.0x1.2mm
Other:
- note added: "Version History -v2.1, Remove the external RTC. There's no need to use an external RTC on the telemetry board. The microcontroller itself has an internal RTC that can be powered from the VBAT line and a 32.768kHz oscillator. Courtesy of Chase! -v2.2, Standardization and cleanup!!"
- note removed: "Version History -v2.1, Remove the external RTC. There's no need to use an external RTC on the telemetry board. The microcontroller itself has an internal RTC that can be powered from the VBAT line and a 32.768kHz oscillator. Courtesy of Chase!"
Changed lines of the file:
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@@
     (stroke (width 0) (type default))
   )
-  (text "Version History\n-v2.1, Remove the external RTC.\nThere's no need to use an external RTC on the telemetry board. The\nmicrocontroller itself has an internal RTC that can be powered from\nthe VBAT line and a 32.768kHz oscillator. Courtesy of Chase!"
+  (text "Version History\n-v2.1, Remove the external RTC.\nThere's no need to use an external RTC on the telemetry board. The\nmicrocontroller itself has an internal RTC that can be powered from\nthe VBAT line and a 32.768kHz oscillator. Courtesy of Chase!\n-v2.2, Standardization and cleanup!!"
     (at 300.99 196.85 0)
     (effects (font (size 2 2)) (justify left bottom))
@@
       (effects (font (size 1.27 1.27)) (justify left))
     )
-    (property "Footprint" "Button_Switch_SMD:SW_SPST_B3SL-1002P" (at 316.865 63.5 0)
+    (property "Footprint" "UTSVT_Special:SW_SPST_B3SL-1002P" (at 316.865 63.5 0)
       (effects (font (size 1.27 1.27)) hide)
     )
@@
       (effects (font (size 1.27 1.27)) (justify left))
     )
-    (property "Footprint" "Crystal:Crystal_SMD_TXC_7A-2Pin_5x3.2mm" (at 156.21 74.93 0)
+    (property "Footprint" "UTSVT_Special:Crystal_SMD_TXC_7A-2Pin_5x3.2mm" (at 156.21 74.93 0)
       (effects (font (size 1.27 1.27)) hide)
     )
@@
       (effects (font (size 1.27 1.27)) (justify left))
     )
-    (property "Footprint" "Button_Switch_SMD:SW_SPST_B3SL-1002P" (at 313.69 111.76 0)
+    (property "Footprint" "UTSVT_Special:SW_SPST_B3SL-1002P" (at 313.69 111.76 0)
       (effects (font (size 1.27 1.27)) hide)
     )
@@
       (effects (font (size 1.27 1.27)) (justify left))
     )
-    (property "Footprint" "Crystal:Crystal_SMD_2012-2Pin_2.0x1.2mm" (at 236.22 179.07 0)
-      (effects (font (size 1.27 1.27)) hide)
-    )
+    (property "Footprint" "UTSVT_Special:Crystal_SMD_2012-2Pin_2.0x1.2mm" (at 236.22 179.07 0)
+      (effects (font (size 1.27 1.27)) hide)
+    )

Commit message: bom, gerbers, edge cuts, footprint verification
Parts:
- BT?: P/N (none) -> 3000TR
- C1, C10, C11, C12, C13, C14, C15, C16, C17, C18, C19, C2, C5, C6, C7, C9: P/N (none) -> C0805C104K5RAC7411
- C20: P/N (none) -> 08055D475KAT2A
- C3, C4: P/N (none) -> 08053A180JAT2A
- C35, C50: P/N (none) -> 08055A9R0JAT2A
- C8: P/N (none) -> 08055C105K4T4A
- H1, H2, H3, H4, LOGO1, LOGO2: P/N (none) -> n/a
- J1, J2, J3, J5, J6: P/N (none) -> 10129378-910001BLF
- R? (x2): P/N (none) -> CRCW08054K70FKEA
- R?: P/N (none) -> CR0805-FX-5490ELF
- U1: P/N (none) -> STM32F429ZIT6
- Y1: P/N 7A-8.000MAHJ-T -> ABM3-8.000MHZ-D2Y-T
- Y3: P/N (none) -> 9HT11-32.768KDZF-T
Other:
- note added: "Load capacitance of ~14.5p"
- note added: "Load capacitance of ~19p"

Commit message: sch and pcb pdfs
Changed lines of the file:
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@@
   )
   (text "Version History\n-v2.1, Remove the external RTC.\nThere's no need to use an external RTC on the telemetry board. The\nmicrocontroller itself has an internal RTC that can be powered from\nthe VBAT line and a 32.768kHz oscillator. Courtesy of Chase!\n-v2.2, Standardization and cleanup!!"
-    (at 300.99 196.85 0)
+    (at 300.355 251.46 0)
     (effects (font (size 2 2)) (justify left bottom))
   )

Commit message: schematic organization
Parts:
- removed J6: SWD, Connector_PinHeader_2.54mm:PinHeader_1x04_P2.54mm_Vertical, symbol Connector_Generic:Conn_01x04
- added J4: SWD, Connector_PinHeader_2.54mm:PinHeader_1x04_P2.54mm_Vertical, symbol Connector_Generic:Conn_01x04
Connections:
- net +3.3V: now also J4.1 (Pin_1)
- net GND: now also J4.4 (Pin_4)
- net SWCLK: now also J4.2 (Pin_2)
- net SWDIO: now also J4.3 (Pin_3)
Other:
- note added: "2.1 - Removes the external RTC. There's no need to use an external RTC on the telemetry board. The microcontroller itself has an internal RTC that can be powered from the VBAT line and a 32.768kHz oscillator. Courtesy of Chase! Future Changes -Add keepout area around RTC clock (prevent noise) -Add impedance matching resistor to Ethernet line -PR Checklist"
- note added: "Flashing pins"
- note added: "NOTE: Isolated +5V and +3.3V. Use GND as local gnd for all board electronic components. Connect GNDPWR when using +12V."
- note added: "Peripherals"
- note added: "Place near pin 25"
- note added: "Place near pin 33"
- note added: "Place near pin 6"
- note added: "STM32 Core"
- note added: "VERSION HISTORY"
- note removed: "Graphics/Logos"
- note removed: "Isolated +5V and +3.3V. Use GND as local gnd for all board electronic components. Connect GNDPWR when using +12V."
- note removed: "Place near pin 22"
- note removed: "Version History -v2.1, Remove the external RTC. There's no need to use an external RTC on the telemetry board. The microcontroller itself has an internal RTC that can be powered from the VBAT line and a 32.768kHz oscillator. Courtesy of Chase! -v2.2, Standardization and cleanup!!"
- moved on the sheet: BT?, C1, C10, C11, C12, C13, C14, C15, C16, C17, C18, C19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

Commit message: bluetooth schematic additions
Connections:
- net SPI4_CLK: now reaches U1.1 (PE2)
- net PA12: now reaches U1.104 (PA12)
- net SPI3_CS: now reaches U1.110 (PA15)
- net SPI3_CLK: now reaches U1.111 (PC10)
- net SPI3_MISO: now reaches U1.112 (PC11)
- net SPI3_MOSI: now reaches U1.113 (PC12)
- net PD0: now reaches U1.114 (PD0)
- net PD1: now reaches U1.115 (PD1)
- net PD2: now reaches U1.116 (PD2)
- net PD3: now reaches U1.117 (PD3)
- net PD4: now reaches U1.118 (PD4)
- net USART2_TX: now reaches U1.119 (PD5)
- net USART2_RX: now reaches U1.122 (PD6)
- net PD7: now reaches U1.123 (PD7)
- net USART6_RX: now reaches U1.124 (PG9)
- net PG10: now reaches U1.125 (PG10)
- net PG12: now reaches U1.127 (PG12)
- net USART6_TX: now reaches U1.129 (PG14)
- net PG15: now reaches U1.132 (PG15)
- net PB3: now reaches U1.133 (PB3)
- net UART8_RX: now reaches U1.141 (PE0)
- net UART8_TX: now reaches U1.142 (PE1)
- net PE3: now reaches U1.2 (PE3)
- net PC0: now reaches U1.26 (PC0)
- net PC2: now reaches U1.28 (PC2)
- net PC3: now reaches U1.29 (PC3)
- net SPI4_CS: now reaches U1.3 (PE4)
- net WKUP: now reaches U1.34 (PA0)
- net PA3: now reaches U1.37 (PA3)
- net SPI4_MISO: now reaches U1.4 (PE5)
- net PA4: now reaches U1.40 (PA4)
- net PA5: now reaches U1.41 (PA5)
- net PA6: now reaches U1.42 (PA6)
- net PB0: now reaches U1.46 (PB0)
- net PB1: now reaches U1.47 (PB1)
- net PB2: now reaches U1.48 (PB2)
- net PF11: now reaches U1.49 (PF11)
- net SPI4_MOSI: now reaches U1.5 (PE6)
- net PF12: now reaches U1.50 (PF12)
- net PF13: now reaches U1.53 (PF13)
- net PF14: now reaches U1.54 (PF14)
- net PF15: now reaches U1.55 (PF15)
- net PG0: now reaches U1.56 (PG0)
- net PG1: now reaches U1.57 (PG1)
- net SPI2_CLK: now reaches U1.69 (PB10)
- net PC13: now reaches U1.7 (PC13)
- net PB11: now reaches U1.70 (PB11)
- net SPI2_CS: now reaches U1.73 (PB12)
- net SPI2_MISO: now reaches U1.75 (PB14)
- net SPI2_MOSI: now reaches U1.76 (PB15)
- net PD10: now reaches U1.79 (PD10)
- net PD11: now reaches U1.80 (PD11)
- net PD12: now reaches U1.81 (PD12)
- net PD13: now reaches U1.82 (PD13)
- net PD14: now reaches U1.85 (PD14)
- net PD15: now reaches U1.86 (PD15)
- net PG2: now reaches U1.87 (PG2)
- net PG3: now reaches U1.88 (PG3)
- net PG4: now reaches U1.89 (PG4)
- net PG5: now reaches U1.90 (PG5)
- net PG6: now reaches U1.91 (PG6)
- net PG7: now reaches U1.92 (PG7)
- net PG8: now reaches U1.93 (PG8)
- net PC6: now reaches U1.96 (PC6)
- net PC7: now reaches U1.97 (PC7)
- net PC8: now reaches U1.98 (PC8)
- net PC9: now reaches U1.99 (PC9)
- net PF0 renamed I2C2_SDA
- net PF1 renamed I2C2_SCL
- no-connect marks 75 -> 71
Other:
- added sheet Bluetooth (Bluetooth.kicad_sch)
- added sheet Breakouts (Breakouts.kicad_sch)
- added sheet Inputs (Inputs.kicad_sch)
- note added: "2.1 - Removes the external RTC. There's no need to use an external RTC on the telemetry board. The microcontroller itself has an internal RTC that can be powered from the VBAT line and a 32.768kHz oscillator. Courtesy of Chase! 2.2 - New IO and Protection - Bluetooth - 4 buttons + 4 switches - SPI break out - GPIO break out - Power protection circuitry Future Changes -Add keepout area around RTC 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"
- note added: "uC TX->CAN TX uC RX->CAN RX"
- note added: "uC TX->IC RX uC RX->IC TX"
- note added: "uC TX->IC RX uC RX->IC TX Baud: 9600"
- note removed: "2.1 - Removes the external RTC. There's no need to use an external RTC on the telemetry board. The microcontroller itself has an internal RTC that can be powered from the VBAT line and a 32.768kHz oscillator. Courtesy of Chase! Future Changes -Add keepout area around RTC clock (prevent noise) -Add impedance matching resistor to Ethernet line -PR Checklist"
- note removed: "Baud: 9600"
- note removed: "uC Tx -> CAN Tx uC Rx -> CAN Rx"
- note removed: "uC Tx -> UART Rx uC Rx -> UART Tx"
- moved on the sheet: BT?, C1, C10, C11, C12, C13, C14, C15, C16, C17, C18, C19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

Commit message: began input/breakout changes
Connections:
- no-connect marks 71 -> 63
Other:
- sheet Inputs ports: added PD15, PG[2..8]; removed none
- note added: "-must figure out pcb layout first -SPI2 is in a more optimal spot -note: SPI2/3 are 22.5 mb/s vs 45 mb/s other ports"
Changed lines of the file:
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@@
   (no_connect (at 211.455 109.855))
   (no_connect (at 211.455 84.455))
-  (no_connect (at 123.825 74.295))
   (no_connect (at 123.825 109.855))
   (no_connect (at 211.455 168.275))
-  (no_connect (at 123.825 81.915))
   (no_connect (at 211.455 86.995))
-  (no_connect (at 123.825 69.215))
   (no_connect (at 211.455 201.295))
   (no_connect (at 123.825 145.415))
@@
   (no_connect (at 123.825 89.535))
   (no_connect (at 123.825 107.315))
-  (no_connect (at 123.825 76.835))
   (no_connect (at 123.825 137.795))
   (no_connect (at 211.455 173.355))
-  (no_connect (at 123.825 71.755))
-  (no_connect (at 211.455 206.375))
   (no_connect (at 123.825 120.015))
   (no_connect (at 211.455 158.115))
@@
   (no_connect (at 123.825 94.615))
   (no_connect (at 123.825 163.195))
-  (no_connect (at 123.825 84.455))
   (no_connect (at 211.455 147.955))
   (no_connect (at 123.825 102.235))
@@
   (no_connect (at 211.455 140.335))
   (no_connect (at 211.455 186.055))
-  (no_connect (at 123.825 79.375))
   (no_connect (at 211.455 150.495))
   (no_connect (at 211.455 153.035))
-  (no_connect (at 211.455 203.835))
   (no_connect (at 123.825 155.575))
   (no_connect (at 123.825 158.115))
@@
   (no_connect (at 211.455 112.395))
   (no_connect (at 211.455 155.575))
+  (no_connect (at 211.455 203.835))
   (no_connect (at 123.825 86.995))
   (no_connect (at 123.825 99.695))
@@
   (no_connect (at 211.455 38.735))
   (no_connect (at 211.455 145.415))
+  (bus_entry (at 121.285 81.915) (size 2.54 2.54)
+    (stroke (width 0) (type default))
+  )
+  (bus_entry (at 121.285 74.295) (size 2.54 2.54)
+    (stroke (width 0) (type default))
+  )
   (bus_entry (at 121.285 178.435) (size 2.54 2.54)
     (stroke (width 0) (type default))
@@
     (stroke (width 0) (type default))
   )
+  (bus_entry (at 121.285 76.835) (size 2.54 2.54)
+    (stroke (width 0) (type default))
+  )
   (bus_entry (at 121.285 165.735) (size 2.54 2.54)
     (stroke (width 0) (type default))
@@
     (stroke (width 0) (type default))
   )
+  (bus_entry (at 121.285 69.215) (size 2.54 2.54)
+    (stroke (width 0) (type default))
+  )
+  (bus_entry (at 121.285 71.755) (size 2.54 2.54)
+    (stroke (width 0) (type default))
+  )
   (bus_entry (at 121.285 175.895) (size 2.54 2.54)
     (stroke (width 0) (type default))
@@
     (stroke (width 0) (type default))
   )
+  (bus_entry (at 121.285 79.375) (size 2.54 2.54)
+    (stroke (width 0) (type default))
+  )
+  (bus_entry (at 121.285 66.675) (size 2.54 2.54)
+    (stroke (width 0) (type default))
+  )
   (bus_entry (at 121.285 183.515) (size 2.54 2.54)
     (stroke (width 0) (type default))
@@
     (stroke (width 0) (type default))
   )
+  (bus (pts (xy 121.285 79.375) (xy 121.285 81.915))
+    (stroke (width 0) (type default))
+  )
   (wire (pts (xy 303.53 35.56) (xy 303.53 38.1))
     (stroke (width 0) (type default))
@@
     (stroke (width 0) (type default))
   )
+  (bus (pts (xy 121.285 76.835) (xy 121.285 79.375))
+    (stroke (width 0) (type default))
+  )
   (wire (pts (xy 123.825 158.115) (xy 137.16 158.115))
     (stroke (width 0) (type default))
@@
     (stroke (width 0) (type default))
   )
+  (bus (pts (xy 121.285 71.755) (xy 121.285 74.295))
+    (stroke (width 0) (type default))
+  )
   (wire (pts (xy 217.17 158.115) (xy 226.06 158.115))
     (stroke (width 0) (type default))
@@
     (stroke (width 0) (type default))
   )
+  (bus (pts (xy 59.055 211.455) (xy 42.545 211.455))
+    (stroke (width 0) (type default))
+  )
   (wire (pts (xy 115.57 53.975) (xy 115.57 55.245))
     (stroke (width 0) (type default))
@@
     (stroke (width 0) (type default))
   )
+  (wire (pts (xy 59.055 208.915) (xy 42.545 208.915))
+    (stroke (width 0) (type default))
+  )
   (wire (pts (xy 170.18 216.535) (xy 170.18 219.075))
     (stroke (width 0) (type default))
@@
     (stroke (width 0) (type default))
   )
+  (bus (pts (xy 121.285 66.675) (xy 121.285 69.215))
+    (stroke (width 0) (type default))
+  )
   (wire (pts (xy 115.57 53.975) (xy 121.92 53.975))
     (stroke (width 0) (type default))
@@
     (stroke (width 0) (type default))
   )
+  (bus (pts (xy 121.285 74.295) (xy 121.285 76.835))
+    (stroke (width 0) (type default))
+  )
   (wire (pts (xy 302.895 52.705) (xy 302.895 56.515))
     (stroke (width 0) (type default))
@@
     (stroke (width 0) (type default))
   )
+  (bus (pts (xy 121.285 69.215) (xy 121.285 71.755))
+    (stroke (width 0) (type default))
+  )
   (bus (pts (xy 121.285 173.355) (xy 121.285 175.895))
     (stroke (width 0) (type default))
@@
     (effects (font (size 1.27 1.27)) (justify left bottom))
   )
-  (text "Load capacitance of ~19p" (at 97.155 70.485 0)
+  (text "Load capacitance of ~19p" (at 96.52 45.72 0)
     (effects (font (size 1.27 1.27)) (justify left bottom))
   )
@@
     (effects (font (size 2.54 2.54) (thickness 0.508) bold) (justify left bottom))
   )
+  (text "-must figure out pcb layout first\n-SPI2 is in a more optimal spot\n-note: SPI2/3 are 22.5 mb/s \n	vs 45 mb/s other ports"
+    (at 44.45 229.235 0)
+    (effects (font (size 1.27 1.27)) (justify left bottom))
+  )
   (text "Load capacitance of ~14.5p" (at 213.36 174.625 0)
     (effects (font (size 1.27 1.27)) (justify left bottom))
@@
     (effects (font (size 1.27 1.27)) (justify right bottom))
   )
+  (label "PG[2..8]" (at 59.055 211.455 180) (fields_autoplaced)
+    (effects (font (size 1.27 1.27)) (justify right bottom))
+  )
   (label "PC8" (at 211.455 145.415 180) (fields_autoplaced)
     (effects (font (size 1.27 1.27)) (justify right bottom))
@@
     (effects (font (size 1.27 1.27)) (justify right bottom))
   )
+  (label "PG[2..8]" (at 121.285 75.565 90) (fields_autoplaced)
+    (effects (font (size 1.27 1.27)) (justify left bottom))
+  )
   (label "PA8" (at 211.455 59.055 180) (fields_autoplaced)
     (effects (font (size 1.27 1.27)) (justify right bottom))
@@
     (effects (font (size 1.27 1.27)) (justify right bottom))
   )
+  (label "PD15" (at 59.055 208.915 180) (fields_autoplaced)
+    (effects (font (size 1.27 1.27)) (justify right bottom))
+  )
   (label "I2C1_SDA" (at 211.455 99.695 180) (fields_autoplaced)
     (effects (font (size 1.27 1.27)) (justify right bottom))
@@
     )
   )
-  (sheet (at 17.145 227.965) (size 25.4 14.605) (fields_autoplaced)
+  (sheet (at 17.145 220.345) (size 25.4 14.605) (fields_autoplaced)
     (stroke (width 0.1524) (type solid))
     (fill (color 0 0 0 0.0000))
-    (property "Sheetname" "Breakouts" (at 17.145 227.2534 0)
+    (property "Sheetname" "Breakouts" (at 17.145 219.6334 0)
       (effects (font (size 1.27 1.27)) (justify left bottom))
     )
-    (property "Sheetfile" "Breakouts.kicad_sch" (at 17.145 243.1546 0)
+    (property "Sheetfile" "Breakouts.kicad_sch" (at 17.145 235.5346 0)
       (effects (font (size 1.27 1.27)) (justify left top))
     )
@@
     )
   )
-  (sheet (at 17.145 206.375) (size 25.4 12.065) (fields_autoplaced)
+  (sheet (at 17.145 207.01) (size 25.4 6.35) (fields_autoplaced)
     (stroke (width 0.1524) (type solid))
     (fill (color 0 0 0 0.0000))
-    (property "Sheetname" "Inputs" (at 17.145 205.6634 0)
+    (property "Sheetname" "Inputs" (at 17.145 206.2984 0)
       (effects (font (size 1.27 1.27)) (justify left bottom))
     )
-    (property "Sheetfile" "Inputs.kicad_sch" (at 17.145 219.0246 0)
+    (property "Sheetfile" "Inputs.kicad_sch" (at 17.145 213.9446 0)
       (effects (font (size 1.27 1.27)) (justify left top))
     )
+    (pin "PD15" input (at 42.545 208.915 0)
+      (effects (font (size 1.27 1.27)) (justify right))
+    )
+    (pin "PG[2..8]" input (at 42.545 211.455 0)
+      (effects (font (size 1.27 1.27)) (justify right))
+    )
     (instances

Commit message: new bt module + preliminary reverse protection
Other:
- note added: "-choose spi breakout based on rearranging everything"
- note added: "2.1 - Removes the external RTC. There's no need to use an external RTC on the telemetry board. The microcontroller itself has an internal RTC that can be powered from the VBAT line and a 32.768kHz oscillator. Courtesy of Chase! 2.2 - New IO and Protection - Bluetooth, never actually tested please research - 4 buttons + 4 switches, hw debouncing - SPI break out, choose best for layout - GPIO break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"
- note removed: "-must figure out pcb layout first -SPI2 is in a more optimal spot -note: SPI2/3 are 22.5 mb/s vs 45 mb/s other ports"
- note removed: "2.1 - Removes the external RTC. There's no need to use an external RTC on the telemetry board. The microcontroller itself has an internal RTC that can be powered from the VBAT line and a 32.768kHz oscillator. Courtesy of Chase! 2.2 - New IO and Protection - Bluetooth - 4 buttons + 4 switches - SPI break out - GPIO break out - Power protection circuitry Future Changes -Add keepout area around RTC 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"
- moved on the sheet: C6, C8
